File: hard/salomon.kicad_sch (KiCad schematic)
At the start: 5 parts

Commit message: Add Hardware en KiCad
Parts:
- removed U?: MAX3232, symbol Interface_UART:MAX3232
- added M?: Shield_D1_mini_DataLogger, symbol Tochi:Shield_D1_mini_DataLogger
- added M?: Shield_D1_mini_DC_Power, symbol Tochi:Shield_D1_mini_DC_Power
Connections:
- net +3V3: now also M?.8 (3V3)
- net GND: now also M?.10 (GND), M?.10 (GND)
- net at J?.1: no longer J?.2
- net at J?.2: no longer J?.3
- net at U?.13 (SDA/D2): now also M?.13 (SDA/D2)
- net at U?.14 (SCL/D1): now also M?.14 (SCL/D1)
- net at U?.4 (SCK/D5): now also M?.4 (D5/SCK)
- net at U?.5 (MISO/D6): now also M?.5 (D6/DO)
- net at U?.6 (MOSI/D7): now also M?.6 (D7/DI)
- net at U?.7 (CS/D8): now also M?.7 (D8/CS)
- net +5V: now reaches U?.9 (5V)
- net +5V: now also M?.9 (5V)
- net +12V: now reaches J?.6
- net +12V: now also M?.0 (Vin)
- net 0V: no longer names the net of J?.4, J?.5
- net 12V: no longer names the net of J?.6, J?.8
Other:
- moved on the sheet: J?, U?
